Commit message: checked

File: base.xacro (robot description, xacro)
@@ -1,153 +1,45 @@
 <?xml version="1.0" ?>
 <!-- =================================================================================== -->
-<!-- |    This document was autogenerated by xacro from src/four_wheel_vehicle/urdf/base.xacro | -->
+<!-- |    This document was autogenerated by xacro from src/four_wheel_vehicle/urdf/base_gazcbo.xacro | -->
 <!-- |    EDITING THIS FILE BY HAND IS NOT RECOMMENDED                                 | -->
 <!-- =================================================================================== -->
 <robot>
-  <material name="blue">
-    <color rgba="0 0 0.5 1"/>
-  </material>
-  <material name="grey">
-    <color rgba="0.5 0.5 0.5 1"/>
-  </material>
-  <material name="orange">
-    <color rgba="1.0 0.5 0 1"/>
-  </material>
-  <material name="yellow">
-    <color rgba="1.0 1.0 0 1"/>
-  </material>
-  <link name="base_footprint"/>
-  <link name="base_link">
-    <visual>
-      <geometry>
-        <box size="0.6 0.4 0.2"/>
-      </geometry>
-      <origin rpy="0 0 0" xyz="0 0 0.1"/>
-      <material name="blue"/>
-    </visual>
-    <collision>
-      <geometry>
-        <box size="0.6 0.4 0.2"/>
-      </geometry>
-      <origin rpy="0 0 0" xyz="0 0 0.1"/>
-    </collision>
-    <inertial>
-      <origin rpy="0 0 0" xyz="0 0 0.1"/>
-      <mass value="5.0"/>
-      <inertia ixx="0.6666666666666667" ixy="0" ixz="0" iyy="0.6666666666666667" iyz="0" izz="0.6666666666666667"/>
-    </inertial>
-  </link>
-  <link name="front_left_wheel_link">
-    <visual>
-      <geometry>
-        <cylinder length="0.05" radius="0.1"/>
-      </geometry>
-      <origin rpy="1.5708 0 0" xyz="0 0 0"/>
-      <material name="grey"/>
-    </visual>
-    <collision>
-      <geometry>
-        <cylinder length="0.05" radius="0.1"/>
-      </geometry>
-      <origin rpy="1.5708 0 0" xyz="0 0 0"/>
-    </collision>
-    <inertial>
-      <origin rpy="1.5708 0 0" xyz="0 0 0"/>
-      <mass value="1.0"/>
-      <inertia ixx="0.010833333333333335" ixy="0" ixz="0" iyy="0.010833333333333335" iyz="0" izz="0.010833333333333335"/>
-    </inertial>
-  </link>
-  <link name="front_right_wheel_link">
-    <visual>
-      <geometry>
-        <cylinder length="0.05" radius="0.1"/>
-      </geometry>
-      <origin rpy="1.5708 0 0" xyz="0 0 0"/>
-      <material name="grey"/>
-    </visual>
-    <collision>
-      <geometry>
-        <cylinder length="0.05" radius="0.1"/>
-      </geometry>
-      <origin rpy="1.5708 0 0" xyz="0 0 0"/>
-    </collision>
-    <inertial>
-      <origin rpy="1.5708 0 0" xyz="0 0 0"/>
-      <mass value="1.0"/>
-      <inertia ixx="0.010833333333333335" ixy="0" ixz="0" iyy="0.010833333333333335" iyz="0" izz="0.010833333333333335"/>
-    </inertial>
-  </link>
-  <link name="rear_left_wheel_link">
-    <visual>
-      <geometry>
-        <cylinder length="0.05" radius="0.1"/>
-      </geometry>
-      <origin rpy="1.5708 0 0" xyz="0 0 0"/>
-      <material name="grey"/>
-    </visual>
-    <collision>
-      <geometry>
-        <cylinder length="0.05" radius="0.1"/>
-      </geometry>
-      <origin rpy="1.5708 0 0" xyz="0 0 0"/>
-    </collision>
-    <inertial>
-      <origin rpy="1.5708 0 0" xyz="0 0 0"/>
-      <mass value="1.0"/>
-      <inertia ixx="0.010833333333333335" ixy="0" ixz="0" iyy="0.010833333333333335" iyz="0" izz="0.010833333333333335"/>
-    </inertial>
-  </link>
-  <link name="rear_right_wheel_link">
-    <visual>
-      <geometry>
-        <cylinder length="0.05" radius="0.1"/>
-      </geometry>
-      <origin rpy="1.5708 0 0" xyz="0 0 0"/>
-      <material name="grey"/>
-    </visual>
-    <collision>
-      <geometry>
-        <cylinder length="0.05" radius="0.1"/>
-      </geometry>
-      <origin rpy="1.5708 0 0" xyz="0 0 0"/>
-    </collision>
-    <inertial>
-      <origin rpy="1.5708 0 0" xyz="0 0 0"/>
-      <mass value="1.0"/>
-      <inertia ixx="0.010833333333333335" ixy="0" ixz="0" iyy="0.010833333333333335" iyz="0" izz="0.010833333333333335"/>
-    </inertial>
-  </link>
-  <joint name="base_joint" type="fixed">
-    <parent link="base_footprint"/>
-    <child link="base_link"/>
-    <origin rpy="0 0 0" xyz="0 0 0.1"/>
-  </joint>
-  <joint name="front_left_wheel_joint" type="revolute">
-    <parent link="base_link"/>
-    <child link="front_left_wheel_link"/>
-    <origin rpy="0 0 0" xyz="0.24 0.225 0"/>
-    <axis xyz="0 1 0"/>
-    <limit effort="100" lower="0" upper="3.14" velocity="10"/>
-  </joint>
-  <joint name="front_right_wheel_joint" type="revolute">
-    <parent link="base_link"/>
-    <child link="front_right_wheel_link"/>
-    <origin rpy="0 0 0" xyz="0.24 -0.225 0"/>
-    <axis xyz="0 1 0"/>
-    <limit effort="100" lower="0" upper="3.14" velocity="10"/>
-  </joint>
-  <joint name="rear_left_wheel_joint" type="revolute">
-    <parent link="base_link"/>
-    <child link="rear_left_wheel_link"/>
-    <origin rpy="0 0 0" xyz="-0.24 0.225 0"/>
-    <axis xyz="0 1 0"/>
-    <limit effort="100" lower="0" upper="3.14" velocity="10"/>
-  </joint>
-  <joint name="rear_right_wheel_joint" type="revolute">
-    <parent link="base_link"/>
-    <child link="rear_right_wheel_link"/>
-    <origin rpy="0 0 0" xyz="-0.24 -0.225 0"/>
-    <axis xyz="0 1 0"/>
-    <limit effort="100" lower="0" upper="3.14" velocity="10"/>
-  </joint>
+  <!-- Malzeme Tanımları -->
+  <gazebo reference="base_link">
+    <material>Gazebo/Blue</material>
+  </gazebo>
+  <gazebo reference="front_left_wheel_link">
+    <material>Gazebo/Grey</material>
+  </gazebo>
+  <gazebo reference="front_right_wheel_link">
+    <material>Gazebo/Grey</material>
+  </gazebo>
+  <gazebo reference="rear_left_wheel_link">
+    <material>Gazebo/Grey</material>
+  </gazebo>
+  <gazebo reference="rear_right_wheel_link">
+    <material>Gazebo/Grey</material>
+  </gazebo>
+  <gazebo>
+    <plugin filename="libgazebo_ros_diff_drive.so" name="diff_drive_controller">
+      <!-- Update rate in Hz -->
+      <update_rate>50</update_rate>
+      <num_wheel__pairs>2</num_wheel__pairs>
+      <!-- wheels -->
+      <left_joint>front_left_wheel_joint</left_joint>
+      <right_joint>front_right_wheel_joint</right_joint>
+      <left_joint>rear_right_wheel_joint</left_joint>
+      <right_joint>rear_wheel_joint</right_joint>
+      <!-- kinematics -->
+      <wheel_separation>0.45</wheel_separation>
+      <wheel_diameter>0.2</wheel_diameter>
+      <!-- output -->
+      <publish_odom>true</publish_odom>
+      <publish_odom_tf>true</publish_odom_tf>
+      <publish_wheel_tf>true</publish_wheel_tf>
+      <odometry_topic>odom</odometry_topic>
+      <odometry_frame>odom</odometry_frame>
+      <robot_base_frame>base_footprint</robot_base_frame>
+    </plugin>
+  </gazebo>
 </robot>

File: install/four_wheel_vehicle/share/four_wheel_vehicle/urdf/base.xacro (robot description, xacro)
@@ -28,31 +28,7 @@
     <xacro:wheel_link prefix = "rear_right"  wheel_mass = "${wheel_mass}" wheel_radius = "${wheel_radius}" wheel_length="${wheel_length}"/>
     <xacro:base_joint/>
-    <joint name="front_left_wheel_joint" type="revolute">
-        <parent link="base_link"/>
-        <child link="front_left_wheel_link"/>
-        <origin xyz="${base_length / 2.5} ${(base_width / 2.0) + (wheel_length / 2.0)} 0" rpy="0 0 0"/>
-        <axis xyz="0 1 0"/>
-        <limit effort="100" velocity="10" lower="0" upper="3.14"/>
-    </joint>
-    <joint name="front_right_wheel_joint" type="revolute">
-        <parent link="base_link"/>
-        <child link="front_right_wheel_link"/>
-        <origin xyz="${base_length / 2.5} -${(base_width / 2.0) + (wheel_length / 2.0)} 0" rpy="0 0 0"/>
-        <axis xyz="0 1 0"/>
-        <limit effort="100" velocity="10" lower="0" upper="3.14"/>
-    </joint>
-    <joint name="rear_left_wheel_joint" type="revolute">
-        <parent link="base_link"/>
-        <child link="rear_left_wheel_link"/>
-        <origin xyz="-${base_length / 2.5} ${(base_width / 2.0) + (wheel_length / 2.0)} 0" rpy="0 0 0"/>
-        <axis xyz="0 1 0"/>
-        <limit effort="100" velocity="10" lower="0" upper="3.14"/>
-    </joint>
-    <joint name="rear_right_wheel_joint" type="revolute">
-        <parent link="base_link"/>
-        <child link="rear_right_wheel_link"/>
-        <origin xyz="-${base_length / 2.5} -${(base_width / 2.0) + (wheel_length / 2.0)} 0" rpy="0 0 0"/>
-        <axis xyz="0 1 0"/>
-        <limit effort="100" velocity="10" lower="0" upper="3.14"/>
-    </joint>
+    <xacro:wheel_joint prefix="front_left" x="${base_length / 2.5}" y="${(base_width / 2.0) + (wheel_length / 2.0)}" z="0"/>
+    <xacro:wheel_joint prefix="front_right" x="${base_length / 2.5}" y="-${(base_width / 2.0) + (wheel_length / 2.0)}" z="0"/>
+    <xacro:wheel_joint prefix="rear_left" x="-${base_length / 2.5}" y="${(base_width / 2.0) + (wheel_length / 2.0)}" z="0"/>
+    <xacro:wheel_joint prefix="rear_right" x="-${base_length / 2.5}" y="-${(base_width / 2.0) + (wheel_length / 2.0)}" z="0"/>
 </robot>

File: install/four_wheel_vehicle/share/four_wheel_vehicle/urdf/base_gazcbo.xacro (robot description, xacro)
@@ -18,15 +18,23 @@
     </gazebo>
     <gazebo>
-        <plugin name="skid_steer_drive_controller" filename="libgazebo_ros_skid_steer_drive.so">
-            <updateRate>100.0</updateRate>
-            <robotNamespace>/four_wheel_vehicle</robotNamespace>
-            <leftFrontJoint>front_left_wheel_joint</leftFrontJoint>
-            <rightFrontJoint>front_right_wheel_joint</rightFrontJoint>
-            <wheelSeparation>0.4</wheelSeparation>  <!-- Tekerlekler arasındaki mesafe -->
-            <wheelDiameter>0.2</wheelDiameter>  <!-- Çap, yarıçapın iki katı -->
-            <robotBaseFrame>base_link</robotBaseFrame>
-            <torque>20</torque>  <!-- Motor torku, ihtiyaç duyulursa ayarlanabilir -->
-            <topicName>cmd_vel</topicName>
-            <broadcastTF>false</broadcastTF>
+        <plugin name="diff_drive_controller" filename="libgazebo_ros_diff_drive.so">
+            <!-- Update rate in Hz -->
+            <update_rate>50</update_rate>
+            <num_wheel_pairs>2</num_wheel_pairs>
+            <!-- wheels -->
+            <left_joint>front_left_wheel_joint</left_joint>
+            <right_joint>front_right_wheel_joint</right_joint>
+            <left_joint>rear_left_wheel_joint</left_joint>
+            <right_joint>rear_right_wheel_joint</right_joint>
+            <!-- kinematics -->
+            <wheel_separation>0.4</wheel_separation>
+            <wheel_diameter>0.2</wheel_diameter>
+            <!-- output -->
+            <publish_odom>true</publish_odom>
+            <publish_odom_tf>true</publish_odom_tf>
+            <publish_wheel_tf>true</publish_wheel_tf>
+            <odometry_topic>odom</odometry_topic>
+            <odometry_frame>odom</odometry_frame>
+            <robot_base_frame>base_footprint</robot_base_frame>
         </plugin>
     </gazebo>

File: install/four_wheel_vehicle/share/four_wheel_vehicle/urdf/common_properties.xacro (robot description, xacro)
@@ -62,11 +62,10 @@
         </joint>
     </xacro:macro>
-    <xacro:macro name = "wheel_joint" params="prefix x y z">
-        <joint name="${prefix}_wheel_joint" type="revolute">
+    <xacro:macro name="wheel_joint" params="prefix x y z">
+        <joint name="${prefix}_wheel_joint" type="continuous">
             <parent link="base_link"/>
             <child link="${prefix}_wheel_link"/>
             <origin xyz="${x} ${y} ${z}" rpy="0 0 0"/>
             <axis xyz="0 1 0"/>
-            <limit effort="100" velocity="10" lower="0" upper="3.14"/>
         </joint>
     </xacro:macro>

File: src/four_wheel_vehicle/urdf/base_gazcbo.xacro (robot description, xacro)
@@ -18,15 +18,23 @@
     </gazebo>
     <gazebo>
-        <plugin name="skid_steer_drive_controller" filename="libgazebo_ros_skid_steer_drive.so">
-            <updateRate>100.0</updateRate>
-            <robotNamespace>/four_wheel_vehicle</robotNamespace>
-            <leftFrontJoint>front_left_wheel_joint</leftFrontJoint>
-            <rightFrontJoint>front_right_wheel_joint</rightFrontJoint>
-            <wheelSeparation>0.4</wheelSeparation>  <!-- Tekerlekler arasındaki mesafe -->
-            <wheelDiameter>0.2</wheelDiameter>  <!-- Çap, yarıçapın iki katı -->
-            <robotBaseFrame>base_link</robotBaseFrame>
-            <torque>20</torque>  <!-- Motor torku, ihtiyaç duyulursa ayarlanabilir -->
-            <topicName>cmd_vel</topicName>
-            <broadcastTF>false</broadcastTF>
+        <plugin name="diff_drive_controller" filename="libgazebo_ros_diff_drive.so">
+            <!-- Update rate in Hz -->
+            <update_rate>50</update_rate>
+            <num_wheel_pairs>2</num_wheel_pairs>
+            <!-- wheels -->
+            <left_joint>front_left_wheel_joint</left_joint>
+            <right_joint>front_right_wheel_joint</right_joint>
+            <left_joint>rear_left_wheel_joint</left_joint>
+            <right_joint>rear_right_wheel_joint</right_joint>
+            <!-- kinematics -->
+            <wheel_separation>0.4</wheel_separation>
+            <wheel_diameter>0.2</wheel_diameter>
+            <!-- output -->
+            <publish_odom>true</publish_odom>
+            <publish_odom_tf>true</publish_odom_tf>
+            <publish_wheel_tf>true</publish_wheel_tf>
+            <odometry_topic>odom</odometry_topic>
+            <odometry_frame>odom</odometry_frame>
+            <robot_base_frame>base_footprint</robot_base_frame>
         </plugin>
     </gazebo>

Commit message: lidar

File: base.xacro (robot description, xacro)
@@ -1,45 +1,75 @@
 <?xml version="1.0" ?>
 <!-- =================================================================================== -->
-<!-- |    This document was autogenerated by xacro from src/four_wheel_vehicle/urdf/base_gazcbo.xacro | -->
+<!-- |    This document was autogenerated by xacro from src/four_wheel_vehicle/urdf/lidar.xacro | -->
 <!-- |    EDITING THIS FILE BY HAND IS NOT RECOMMENDED                                 | -->
 <!-- =================================================================================== -->
 <robot>
-  <!-- Malzeme Tanımları -->
-  <gazebo reference="base_link">
-    <material>Gazebo/Blue</material>
-  </gazebo>
-  <gazebo reference="front_left_wheel_link">
-    <material>Gazebo/Grey</material>
-  </gazebo>
-  <gazebo reference="front_right_wheel_link">
-    <material>Gazebo/Grey</material>
-  </gazebo>
-  <gazebo reference="rear_left_wheel_link">
-    <material>Gazebo/Grey</material>
-  </gazebo>
-  <gazebo reference="rear_right_wheel_link">
-    <material>Gazebo/Grey</material>
-  </gazebo>
-  <gazebo>
-    <plugin filename="libgazebo_ros_diff_drive.so" name="diff_drive_controller">
-      <!-- Update rate in Hz -->
-      <update_rate>50</update_rate>
-      <num_wheel__pairs>2</num_wheel__pairs>
-      <!-- wheels -->
-      <left_joint>front_left_wheel_joint</left_joint>
-      <right_joint>front_right_wheel_joint</right_joint>
-      <left_joint>rear_right_wheel_joint</left_joint>
-      <right_joint>rear_wheel_joint</right_joint>
-      <!-- kinematics -->
-      <wheel_separation>0.45</wheel_separation>
-      <wheel_diameter>0.2</wheel_diameter>
-      <!-- output -->
-      <publish_odom>true</publish_odom>
-      <publish_odom_tf>true</publish_odom_tf>
-      <publish_wheel_tf>true</publish_wheel_tf>
-      <odometry_topic>odom</odometry_topic>
-      <odometry_frame>odom</odometry_frame>
-      <robot_base_frame>base_footprint</robot_base_frame>
-    </plugin>
+  <link name="lidar_link">
+    <visual>
+      <geometry>
+        <cylinder length="0.05" radius="0.1"/>
+      </geometry>
+      <origin rpy="0 0 0" xyz="0 0 0"/>
+    </visual>
+    <collision>
+      <geometry>
+        <cylinder length="0.05" radius="0.1"/>
+      </geometry>
+      <origin rpy="0 0 0" xyz="0 0 0"/>
+    </collision>
+    <inertial>
+      <origin rpy="0 0 0" xyz="0 0 0"/>
+      <mass value="1.0"/>
+      <inertia ixx="0.002708333333333334" ixy="0" ixz="0" iyy="0.002708333333333334" iyz="0" izz="0.002708333333333334"/>
+    </inertial>
+  </link>
+  <joint name="lidar_base_joint" type="fixed">
+    <origin rpy="0 0 0" xyz="0 0 0.25"/>
+    <parent link="base_link"/>
+    <child link="lidar_link"/>
+  </joint>
+  <gazebo reference="lidar_link">
+    <material>Gazebo/Orange</material>
+    <sensor name="head_hokuyo_sensor" type="ray">
+      <visualize>true</visualize>
+      <update_rate>10</update_rate>
+      <ray>
+        <scan>
+          <horizontal>
+            <samples>181</samples>
+            <resolution>1</resolution>
+            <min_angle>-1.046666667</min_angle>
+            <max_angle>1.04666667</max_angle>
+          </horizontal>
+        </scan>
+        <range>
+          <min>0.08</min>
+          <max>6.0</max>
+          <resolution>0.05</resolution>
+        </range>
+        <noise>
+          <type>gaussian</type>
+          <mean>0.0</mean>
+          <stddev>0.01</stddev>
+        </noise>
+      </ray>
+      <plugin filename="libgazebo_ros_ray_sensor.so" name="lidar_scan">
+        <robotNamespace>/four_wheel_vehicle</robotNamespace>
+        <noise>
+          <type>gaussian</type>
+          <mean>0.0</mean>
+          <stddev>0.01</stddev>
+        </noise>
+        <alwaysOn>true</alwaysOn>
+        <updateRate>30</updateRate>
+        <topicName>/scan</topicName>
+        <frameName>lidar</frameName>
+        <ros>
+          <!-- Ensure that the output topic is correctly remapped -->
+          <remapping>~/out:=/scan</remapping>
+          <outputType>sensor_msgs/PointCloud2</outputType>
+        </ros>
+      </plugin>
+    </sensor>
   </gazebo>
 </robot>

File: install/four_wheel_vehicle/share/four_wheel_vehicle/urdf/vehicle.urdf.xacro (robot description, xacro)
@@ -5,3 +5,4 @@
     <xacro:include filename = "/home/tayya/four_wheel_ws/src/four_wheel_vehicle/urdf/camera.xacro"/>
     <xacro:include filename = "/home/tayya/four_wheel_ws/src/four_wheel_vehicle/urdf/base_gazcbo.xacro"/>
+    <xacro:include filename = "/home/tayya/four_wheel_ws/src/four_wheel_vehicle/urdf/lidar.xacro"/>
 </robot>
