Commit message: a

File: install/four_wheel_vehicle/share/four_wheel_vehicle/urdf/base.xacro (robot description, xacro)
@@ -1,4 +1,5 @@
 <?xml version="1.0"?>
 <robot xmlns:xacro="http://www.ros.org/wiki/xacro">
+    <xacro:include filename = "/home/tayya/four_wheel_ws/src/four_wheel_vehicle/urdf/common_properties.xacro"/>
     <xacro:property name="base_mass" value="5.0"/>
     <xacro:property name="base_length" value="0.6" />
@@ -21,5 +22,5 @@
     </material>
     <link name="base_footprint"/>
-    <xacro:base_link base_mass="${base_mass}" base_length = "${base_length}" base_width = "${base_width}" base_height = "${base_height}"/>
+    <xacro:base_macro base_mass="${base_mass}" base_length = "${base_length}" base_width = "${base_width}" base_height = "${base_height}"/>
     <xacro:wheel_link prefix = "front_left"  wheel_mass = "${wheel_mass}" wheel_radius = "${wheel_radius}" wheel_length="${wheel_length}"/>
     <xacro:wheel_link prefix = "front_right" wheel_mass = "${wheel_mass}" wheel_radius = "${wheel_radius}" wheel_length="${wheel_length}"/>
@@ -27,7 +28,31 @@
     <xacro:wheel_link prefix = "rear_right"  wheel_mass = "${wheel_mass}" wheel_radius = "${wheel_radius}" wheel_length="${wheel_length}"/>
     <xacro:base_joint/>
-    <xacro:wheel_joint prefix = "front_left"  x = "${base_length / 2.0}"  y = "${base_width / 2.0}"  z = "0"/>
-    <xacro:wheel_joint prefix = "front_right" x = "${base_length / 2.0}"  y = "-${base_width / 2.0}" z = "0"/>
-    <xacro:wheel_joint prefix = "rear_left"   x = "-${base_length / 2.0}" y = "${base_width / 2.0}"  z = "0"/>
-    <xacro:wheel_joint prefix = "rear_right"  x = "-${base_length / 2.0}" y = "-${base_width / 2.0}" z = "0"/>
+    <joint name="front_left_wheel_joint" type="revolute">
+        <parent link="base_link"/>
+        <child link="front_left_wheel_link"/>
+        <origin xyz="${base_length / 2.5} ${(base_width / 2.0) + (wheel_length / 2.0)} 0" rpy="0 0 0"/>
+        <axis xyz="0 1 0"/>
+        <limit effort="100" velocity="10" lower="0" upper="3.14"/>
+    </joint>
+    <joint name="front_right_wheel_joint" type="revolute">
+        <parent link="base_link"/>
+        <child link="front_right_wheel_link"/>
+        <origin xyz="${base_length / 2.5} -${(base_width / 2.0) + (wheel_length / 2.0)} 0" rpy="0 0 0"/>
+        <axis xyz="0 1 0"/>
+        <limit effort="100" velocity="10" lower="0" upper="3.14"/>
+    </joint>
+    <joint name="rear_left_wheel_joint" type="revolute">
+        <parent link="base_link"/>
+        <child link="rear_left_wheel_link"/>
+        <origin xyz="-${base_length / 2.5} ${(base_width / 2.0) + (wheel_length / 2.0)} 0" rpy="0 0 0"/>
+        <axis xyz="0 1 0"/>
+        <limit effort="100" velocity="10" lower="0" upper="3.14"/>
+    </joint>
+    <joint name="rear_right_wheel_joint" type="revolute">
+        <parent link="base_link"/>
+        <child link="rear_right_wheel_link"/>
+        <origin xyz="-${base_length / 2.5} -${(base_width / 2.0) + (wheel_length / 2.0)} 0" rpy="0 0 0"/>
+        <axis xyz="0 1 0"/>
+        <limit effort="100" velocity="10" lower="0" upper="3.14"/>
+    </joint>
 </robot>

File: install/four_wheel_vehicle/share/four_wheel_vehicle/urdf/base_gazcbo.xacro (robot description, xacro)
@@ -1,36 +1,32 @@
 <?xml version="1.0"?>
 <robot xmlns:xacro="http://www.ros.org/wiki/xacro">
-    <gazebo reference = "base_link">
+    <!-- Malzeme Tanımları -->
+    <gazebo reference="base_link">
         <material>Gazebo/Blue</material>
     </gazebo>
-    <gazebo reference = "front_left_wheel_link">
+    <gazebo reference="front_left_wheel_link">
         <material>Gazebo/Grey</material>
     </gazebo>
-    <gazebo reference = "front_right_wheel_link">
+    <gazebo reference="front_right_wheel_link">
         <material>Gazebo/Grey</material>
     </gazebo>
-    <gazebo reference = "rear_left_wheel_link">
+    <gazebo reference="rear_left_wheel_link">
         <material>Gazebo/Grey</material>
     </gazebo>
-    <gazebo reference = "rear_right_wheel_link">
+    <gazebo reference="rear_right_wheel_link">
         <material>Gazebo/Grey</material>
     </gazebo>
     <gazebo>
-        <plugin name="diff_drive_controller" filename="libgazebo_ros_diff_drive.so">
-            <!-- Update rate in Hz -->
-            <update_rate>50</update_rate>
-            <!-- wheels -->
-            <left_joint>left_wheel_joint</left_joint>
-            <right_joint>right_wheel_joint</right_joint>
-            <!-- kinematics -->
-            <wheel_separation>0.45</wheel_separation>
-            <wheel_diameter>0.2</wheel_diameter>
-            <!-- output -->
-            <publish_odom>true</publish_odom>
-            <publish_odom_tf>true</publish_odom_tf>
-            <publish_wheel_tf>true</publish_wheel_tf>
-            <odometry_topic>odom</odometry_topic>
-            <odometry_frame>odom</odometry_frame>
-            <robot_base_frame>base_footprint</robot_base_frame>
+        <plugin name="skid_steer_drive_controller" filename="libgazebo_ros_skid_steer_drive.so">
+            <updateRate>100.0</updateRate>
+            <robotNamespace>/four_wheel_vehicle</robotNamespace>
+            <leftFrontJoint>front_left_wheel_joint</leftFrontJoint>
+            <rightFrontJoint>front_right_wheel_joint</rightFrontJoint>
+            <wheelSeparation>0.4</wheelSeparation>  <!-- Tekerlekler arasındaki mesafe -->
+            <wheelDiameter>0.2</wheelDiameter>  <!-- Çap, yarıçapın iki katı -->
+            <robotBaseFrame>base_link</robotBaseFrame>
+            <torque>20</torque>  <!-- Motor torku, ihtiyaç duyulursa ayarlanabilir -->
+            <topicName>cmd_vel</topicName>
+            <broadcastTF>false</broadcastTF>
         </plugin>
     </gazebo>

File: install/four_wheel_vehicle/share/four_wheel_vehicle/urdf/camera.xacro (robot description, xacro)
@@ -16,9 +16,10 @@
             </geometry>
         </collision>
+        <xacro:box_inertia  m="0.1" l="${camera_length}" w = "${camera_width}" h= "${camera_height}"  xyz="0 0 0" rpy="0 0 0"/>
     </link>
     <joint name = "base_camera_joint" type = "fixed">
         <parent link = "base_link"/>
         <child link = "camera_link"/>
-        <origin xyz = "${(base_length + camera_length) / 2.0} 0 ${base_height /2}" rpy = "0 0 0"/>
+        <origin xyz = "${(base_length + camera_length) / 2.0} 0 ${base_height-(camera_height/2.0)}" rpy = "0 0 0"/>
     </joint>
     <gazebo reference = "camera_link">

File: install/four_wheel_vehicle/share/four_wheel_vehicle/urdf/common_properties.xacro (robot description, xacro)
@@ -1,5 +1,5 @@
 <?xml version="1.0"?>
 <robot xmlns:xacro="http://www.ros.org/wiki/xacro">
-    <xacro:macro name = "base_link" params="base_mass base_length base_width base_height">
+    <xacro:macro name = "base_macro" params="base_mass base_length base_width base_height">
         <link name="base_link">
             <visual>
@@ -16,13 +16,5 @@
                 <origin xyz="0 0 ${base_height / 2.0}" rpy="0 0 0"/>
             </collision>
-            <inertial>
-                <origin xyz="0 0 ${base_height / 2.0}" rpy="0 0 0"/>
-                <mass value="${base_mass}"/>
-                <inertia ixx="${base_mass * (base_width * base_width + base_height * base_height) / 12}"
-                        ixy="0" ixz="0"
-                        iyy="${base_mass * (base_length * base_length + base_height * base_height) / 12}"
-                        iyz="0"
-                        izz="${base_mass * (base_length * base_length + base_width * base_width) / 12}"/>
-            </inertial>
+            <xacro:box_inertia m="5.0" l="${2*base_length}" w="${2*base_width}" h="${2*base_height}" xyz="0 0 ${base_height / 2.0}" rpy="0 0 0"/>
         </link>
     </xacro:macro>
@@ -42,20 +34,15 @@
                 <origin xyz="0 0 0" rpy="1.5708 0 0"/>
             </collision>
-            <inertial>
-                <mass value="${wheel_mass}"/>
-                <inertia ixx="${(wheel_mass / 12) * (3 * wheel_radius * wheel_radius + wheel_length * wheel_length)}"
-                        ixy="0" ixz="0"
-                        iyy="${(wheel_mass / 12) * (3 * wheel_radius * wheel_radius + wheel_length * wheel_length)}"
-                        iyz="0"
-                        izz="${(wheel_mass / 12) * (3 * wheel_radius * wheel_radius + wheel_length * wheel_length)}"/>
-            </inertial>
+            <xacro:wheel_inertia m = "1.0" r = "${2*wheel_radius}" h = "${2*wheel_length}" xyz="0 0 0" rpy="1.5708 0 0"/>
         </link>
     </xacro:macro>
-    <xacro:macro name = "base_inertia" params="mass x y z">
-        <mass value = "${mass}" />
-        <inertia
-            ixx="${mass * (y*y + z*z) / 12}"
-            iyy="${mass * (x*x + z*z) / 12}"
-            izz="${mass * (x*x + y*y) / 12}" />
+    <xacro:macro name = "box_inertia" params = "m l w h xyz rpy">
+        <inertial>
+            <origin xyz = "${xyz}" rpy = "${rpy}" />
+            <mass value = "${m}" />
+            <inertia ixx = "${(m/12) * (l*l+h*h)}" ixy = "0" ixz = "0"
+            iyy = "${(m/12) * (l*l+h*h)}" iyz = "0"
+            izz = "${(m/12) * (l*l+h*h)}"/>
+        </inertial>
     </xacro:macro>
     <xacro:macro name = "wheel_inertia" params = "m r h xyz rpy">
@@ -76,9 +63,10 @@
     </xacro:macro>
     <xacro:macro name = "wheel_joint" params="prefix x y z">
-        <joint name="${prefix}_wheel_joint" type="continuous">
+        <joint name="${prefix}_wheel_joint" type="revolute">
             <parent link="base_link"/>
             <child link="${prefix}_wheel_link"/>
             <origin xyz="${x} ${y} ${z}" rpy="0 0 0"/>
             <axis xyz="0 1 0"/>
+            <limit effort="100" velocity="10" lower="0" upper="3.14"/>
         </joint>
     </xacro:macro>

File: src/four_wheel_vehicle/urdf/base_gazcbo.xacro (robot description, xacro)
@@ -1,36 +1,32 @@
 <?xml version="1.0"?>
 <robot xmlns:xacro="http://www.ros.org/wiki/xacro">
-    <gazebo reference = "base_link">
+    <!-- Malzeme Tanımları -->
+    <gazebo reference="base_link">
         <material>Gazebo/Blue</material>
     </gazebo>
-    <gazebo reference = "front_left_wheel_link">
+    <gazebo reference="front_left_wheel_link">
         <material>Gazebo/Grey</material>
     </gazebo>
-    <gazebo reference = "front_right_wheel_link">
+    <gazebo reference="front_right_wheel_link">
         <material>Gazebo/Grey</material>
     </gazebo>
-    <gazebo reference = "rear_left_wheel_link">
+    <gazebo reference="rear_left_wheel_link">
         <material>Gazebo/Grey</material>
     </gazebo>
-    <gazebo reference = "rear_right_wheel_link">
+    <gazebo reference="rear_right_wheel_link">
         <material>Gazebo/Grey</material>
     </gazebo>
     <gazebo>
-        <plugin name="diff_drive_controller" filename="libgazebo_ros_diff_drive.so">
-            <!-- Update rate in Hz -->
-            <update_rate>50</update_rate>
-            <!-- wheels -->
-            <left_joint>left_wheel_joint</left_joint>
-            <right_joint>right_wheel_joint</right_joint>
-            <!-- kinematics -->
-            <wheel_separation>0.45</wheel_separation>
-            <wheel_diameter>0.2</wheel_diameter>
-            <!-- output -->
-            <publish_odom>true</publish_odom>
-            <publish_odom_tf>true</publish_odom_tf>
-            <publish_wheel_tf>true</publish_wheel_tf>
-            <odometry_topic>odom</odometry_topic>
-            <odometry_frame>odom</odometry_frame>
-            <robot_base_frame>base_footprint</robot_base_frame>
+        <plugin name="skid_steer_drive_controller" filename="libgazebo_ros_skid_steer_drive.so">
+            <updateRate>100.0</updateRate>
+            <robotNamespace>/four_wheel_vehicle</robotNamespace>
+            <leftFrontJoint>front_left_wheel_joint</leftFrontJoint>
+            <rightFrontJoint>front_right_wheel_joint</rightFrontJoint>
+            <wheelSeparation>0.4</wheelSeparation>  <!-- Tekerlekler arasındaki mesafe -->
+            <wheelDiameter>0.2</wheelDiameter>  <!-- Çap, yarıçapın iki katı -->
+            <robotBaseFrame>base_link</robotBaseFrame>
+            <torque>20</torque>  <!-- Motor torku, ihtiyaç duyulursa ayarlanabilir -->
+            <topicName>cmd_vel</topicName>
+            <broadcastTF>false</broadcastTF>
         </plugin>
     </gazebo>

Commit message: _

File: install/four_wheel_vehicle/share/four_wheel_vehicle/urdf/base.xacro (robot description, xacro)
@@ -9,4 +9,8 @@
     <xacro:property name="wheel_radius" value="0.1" />
     <xacro:property name="wheel_length" value="0.05" />
+    <xacro:property name="holder_mass" value="1.0" />
+    <xacro:property name="holder_x" value="0.2" />
+    <xacro:property name="holder_y" value="0.05" />
+    <xacro:property name="holder_z" value="0.05" />
     <material name="blue">
         <color rgba="0 0 0.5 1"/>
@@ -23,12 +27,20 @@
     <link name="base_footprint"/>
     <xacro:base_macro base_mass="${base_mass}" base_length = "${base_length}" base_width = "${base_width}" base_height = "${base_height}"/>
+    <xacro:base_joint/>
+    <xacro:wheel_holder_link_xacro prefix="front_left" holder_mass="${holder_mass}" holder_x="${holder_x}" holder_y="${holder_y}" holder_z="${holder_z}"/>
+    <xacro:wheel_holder_link_xacro prefix="front_right" holder_mass="${holder_mass}" holder_x="${holder_x}" holder_y="${holder_y}" holder_z="${holder_z}"/>
+    <xacro:wheel_holder_link_xacro prefix="rear_left" holder_mass="${holder_mass}" holder_x="${holder_x}" holder_y="${holder_y}" holder_z="${holder_z}"/>
+    <xacro:wheel_holder_link_xacro prefix="rear_right" holder_mass="${holder_mass}" holder_x="${holder_x}" holder_y="${holder_y}" holder_z="${holder_z}"/>
     <xacro:wheel_link prefix = "front_left"  wheel_mass = "${wheel_mass}" wheel_radius = "${wheel_radius}" wheel_length="${wheel_length}"/>
     <xacro:wheel_link prefix = "front_right" wheel_mass = "${wheel_mass}" wheel_radius = "${wheel_radius}" wheel_length="${wheel_length}"/>
     <xacro:wheel_link prefix = "rear_left"   wheel_mass = "${wheel_mass}" wheel_radius = "${wheel_radius}" wheel_length="${wheel_length}"/>
     <xacro:wheel_link prefix = "rear_right"  wheel_mass = "${wheel_mass}" wheel_radius = "${wheel_radius}" wheel_length="${wheel_length}"/>
-    <xacro:base_joint/>
-    <xacro:wheel_joint prefix="front_left" x="${base_length / 2.5}" y="${(base_width / 2.0) + (wheel_length / 2.0)}" z="0"/>
-    <xacro:wheel_joint prefix="front_right" x="${base_length / 2.5}" y="-${(base_width / 2.0) + (wheel_length / 2.0)}" z="0"/>
-    <xacro:wheel_joint prefix="rear_left" x="-${base_length / 2.5}" y="${(base_width / 2.0) + (wheel_length / 2.0)}" z="0"/>
-    <xacro:wheel_joint prefix="rear_right" x="-${base_length / 2.5}" y="-${(base_width / 2.0) + (wheel_length / 2.0)}" z="0"/>
+    <xacro:wheel_holder_joint prefix="front_left" x="0.3" y="0.2" z="-0.1"/>
+    <xacro:wheel_holder_joint prefix="front_right" x="0.3" y="-0.2" z="-0.1"/>
+    <xacro:wheel_holder_joint prefix="rear_left" x="-0.3" y="0.2" z="-0.1"/>
+    <xacro:wheel_holder_joint prefix="rear_right" x="-0.3" y="-0.2" z="-0.1"/>
+    <xacro:wheel_joint prefix="front_left" x="0.1" y="${holder_z}" z="0.0"/>
+    <xacro:wheel_joint prefix="front_right" x="0.1" y="${-holder_z}" z="0.0"/>
+    <xacro:wheel_joint prefix="rear_left" x="0.1" y="${holder_z}" z="0.0"/>
+    <xacro:wheel_joint prefix="rear_right" x="0.1" y="${-holder_z}" z="0.0"/>
 </robot>

File: install/four_wheel_vehicle/share/four_wheel_vehicle/urdf/base_gazcbo.xacro (robot description, xacro)
@@ -1,5 +1,4 @@
 <?xml version="1.0"?>
 <robot xmlns:xacro="http://www.ros.org/wiki/xacro">
-    <!-- Malzeme Tanımları -->
     <gazebo reference="base_link">
         <material>Gazebo/Blue</material>
@@ -17,25 +16,31 @@
         <material>Gazebo/Grey</material>
     </gazebo>
+    <gazebo reference="front_left_wheel_holder_link">
+        <material>Gazebo/Orange</material>
+    </gazebo>
+    <gazebo reference="front_right_wheel_holder_link">
+        <material>Gazebo/Orange</material>
+    </gazebo>
+    <gazebo reference="rear_left_wheel_holder_link">
+        <material>Gazebo/Orange</material>
+    </gazebo>
+    <gazebo reference="rear_right_wheel_holder_link">
+        <material>Gazebo/Orange</material>
+    </gazebo>
     <gazebo>
-        <plugin name="diff_drive_controller" filename="libgazebo_ros_diff_drive.so">
-            <!-- Update rate in Hz -->
-            <update_rate>50</update_rate>
-            <num_wheel_pairs>2</num_wheel_pairs>
-            <!-- wheels -->
-            <left_joint>front_left_wheel_joint</left_joint>
-            <right_joint>front_right_wheel_joint</right_joint>
-            <left_joint>rear_left_wheel_joint</left_joint>
-            <right_joint>rear_right_wheel_joint</right_joint>
-            <!-- kinematics -->
-            <wheel_separation>0.4</wheel_separation>
-            <wheel_diameter>0.2</wheel_diameter>
-            <!-- output -->
-            <publish_odom>true</publish_odom>
-            <publish_odom_tf>true</publish_odom_tf>
-            <publish_wheel_tf>true</publish_wheel_tf>
-            <odometry_topic>odom</odometry_topic>
-            <odometry_frame>odom</odometry_frame>
-            <robot_base_frame>base_footprint</robot_base_frame>
-        </plugin>
+    <plugin name="skid_steer_drive_controller" filename="libgazebo_ros_skid_steer_drive.so">
+        <updateRate>100.0</updateRate>
+        <robotNamespace>/</robotNamespace>
+        <leftFrontJoint>front_left_wheel_joint</leftFrontJoint>
+        <rightFrontJoint>front_right_wheel_joint</rightFrontJoint>
+        <leftRearJoint>rear_left_wheel_joint</leftRearJoint>
+        <rightRearJoint>rear_right_wheel_joint</rightRearJoint>
+        <wheelSeparation>0.4</wheelSeparation>
+        <wheelDiameter>0.215</wheelDiameter>
+        <robotBaseFrame>base_link</robotBaseFrame>
+        <torque>20</torque>
+        <topicName>cmd_vel</topicName>
+        <broadcastTF>false</broadcastTF>
+    </plugin>
     </gazebo>
 </robot>

File: install/four_wheel_vehicle/share/four_wheel_vehicle/urdf/common_properties.xacro (robot description, xacro)
@@ -17,4 +17,22 @@
             </collision>
             <xacro:box_inertia m="5.0" l="${2*base_length}" w="${2*base_width}" h="${2*base_height}" xyz="0 0 ${base_height / 2.0}" rpy="0 0 0"/>
+        </link>
+    </xacro:macro>
+    <xacro:macro name="wheel_holder_link_xacro" params="prefix holder_mass holder_x holder_y holder_z">
+        <link name="${prefix}_wheel_holder_link">
+            <visual>
+                <geometry>
+                    <box size="${holder_x} ${holder_y} ${holder_z}"/>
+                </geometry>
+                <origin xyz="0 0 0" rpy="0 0 0"/>
+                <material name="blue"/>
+            </visual>
+            <collision>
+                <geometry>
+                    <box size="${holder_x} ${holder_y} ${holder_z}"/>
+                </geometry>
+                <origin xyz="0 0 0" rpy="0 0 0"/>
+            </collision>
+            <xacro:box_inertia m="${holder_mass}" l="${holder_x}" w="${holder_y}" h="${holder_z}" xyz="0 0 ${holder_z}" rpy="0 0 0"/>
         </link>
     </xacro:macro>
@@ -59,10 +77,17 @@
             <parent link="base_footprint"/>
             <child link="base_link"/>
-            <origin xyz="0 0 ${wheel_radius}" rpy="0 0 0"/>
+            <origin xyz="0 0 ${wheel_radius + holder_x}" rpy="0 0 0"/>
+        </joint>
+    </xacro:macro>
+    <xacro:macro name="wheel_holder_joint" params="prefix x y z">
+        <joint name="${prefix}_wheel_holder_joint" type="continuous">
+            <parent link="base_link"/>
+            <child link="${prefix}_wheel_holder_link"/>
+            <origin xyz="${x} ${y} ${z}" rpy="0 1.570796325 0"/>
         </joint>
     </xacro:macro>
     <xacro:macro name="wheel_joint" params="prefix x y z">
         <joint name="${prefix}_wheel_joint" type="continuous">
-            <parent link="base_link"/>
+            <parent link="${prefix}_wheel_holder_link"/>
             <child link="${prefix}_wheel_link"/>
             <origin xyz="${x} ${y} ${z}" rpy="0 0 0"/>

File: install/four_wheel_vehicle/share/four_wheel_vehicle/urdf/lidar.xacro (robot description, xacro)
@@ -29,5 +29,5 @@
          <sensor name="laser" type="ray">
             <pose> 0 0 0.25 0 0 0 </pose>
-            <visualize>true</visualize>
+            <visualize>false</visualize>
             <update_rate>10</update_rate>
             <ray>

File: install/four_wheel_vehicle/share/four_wheel_vehicle/urdf/vehicle.urdf.xacro (robot description, xacro)
@@ -3,6 +3,4 @@
     <xacro:include filename = "/home/tayya/four_wheel_ws/src/four_wheel_vehicle/urdf/common_properties.xacro"/>
     <xacro:include filename = "/home/tayya/four_wheel_ws/src/four_wheel_vehicle/urdf/base.xacro"/>
-    <xacro:include filename = "/home/tayya/four_wheel_ws/src/four_wheel_vehicle/urdf/camera.xacro"/>
     <xacro:include filename = "/home/tayya/four_wheel_ws/src/four_wheel_vehicle/urdf/base_gazcbo.xacro"/>
-    <xacro:include filename = "/home/tayya/four_wheel_ws/src/four_wheel_vehicle/urdf/lidar.xacro"/>
 </robot>
